File: hardware/power_system.kicad_sch (KiCad schematic)
At the start: 0 parts

Commit message: finished schematic
Parts:
- added BT201: Battery, symbol Device:Battery_Cell
- added C201: 2.2u, Capacitor_SMD:C_0603_1608Metric, symbol Device:C
- added C202, C203, C204, C205: 1u, Capacitor_SMD:C_0603_1608Metric, symbol Device:C
- added C206, C208, C210: 4.7u, Capacitor_SMD:C_0603_1608Metric, symbol Device:C
- added C207: 10u, Capacitor_SMD:C_0603_1608Metric, symbol Device:C
- added C209: 4.7p, Capacitor_SMD:C_0603_1608Metric, symbol Device:C
- added D201: STPS0530Z, Diode_SMD:D_SOD-123, symbol Device:D
- added F201: VBUS Polyfuse, Fuse:Fuse_1206_3216Metric_Pad1.42x1.75mm_HandSolder, symbol Device:Polyfuse
- added J201: Battery Connector, picowy_footprints:CONN_DF65-3P-1.7V21_HIR, symbol Connector_Generic:Conn_01x02
- added J202: USB_C_Receptacle_USB2.0_14P, picowy_footprints:CONN_124018612112A_AMP, symbol Connector:USB_C_Receptacle_USB2.0_14P
- added L201: 6.8u, Inductor_SMD:L_1210_3225Metric_Pad1.42x2.65mm_HandSolder, symbol Device:L
- added Q201: PMOS, Package_TO_SOT_SMD:SOT-23-3, symbol Simulation_SPICE:PMOS
- added R201: 10m, Resistor_SMD:R_0603_1608Metric, symbol Device:R
- added R202, R207, R210, R211: 10k, Resistor_SMD:R_0603_1608Metric, symbol Device:R
- added R203, R204: 5.1k, Resistor_SMD:R_0603_1608Metric, symbol Device:R
- added R205: 17.4k, Resistor_SMD:R_0603_1608Metric, symbol Device:R
- added R206: 30k, Resistor_SMD:R_0603_1608Metric, symbol Device:R
- added R208: 1.8M, Resistor_SMD:R_0603_1608Metric, symbol Device:R
- added R209: 205k, Resistor_SMD:R_0603_1608Metric, symbol Device:R
- added U201: USBLC6-2SC6, Package_TO_SOT_SMD:SOT-23-6, symbol Power_Protection:USBLC6-2SC6
- added U202: BQ27426, Package_BGA:Texas_DSBGA-9_1.62x1.58mm_Layout3x3_P0.5mm, symbol picowy_symbols:BQ27426
- added U203: TPS7A20xxxDBV, Package_TO_SOT_SMD:SOT-23-5, symbol Regulator_Linear:TPS7A20xxxDBV
- added U204: BQ24230RGT, Package_DFN_QFN:VQFN-16-1EP_3x3mm_P0.5mm_EP1.68x1.68mm_ThermalVias, symbol Power_Management:BQ24230RGT
- added U205: TPS61040DDC, Package_TO_SOT_SMD:SOT-23-5, symbol Regulator_Switching:TPS61040DDC
Connections:
- new net: R207.1, U204.1 (TS)
- new net: R206.2, U204.14 (TMR)
- new net: R205.2, U204.16 (ISET)
- new net +12V: C209.1, C210.1, D201.1 (K), R208.1
- new net +3V3: C205.1, Q201.3 (S), R210.1, R211.1, U203.5 (OUT)
- new net +BATT: C204.1, J201.2 (Pin_2), R201.2, U202.C1 (SRP), U202.C3 (BAT)
- new net 12V_FB: C209.2, R208.2, R209.1, U205.3 (FB)
- new net 12V_SW: D201.2 (A), L201.2, U205.1 (SW)
- new net BATT_IN: C206.1, R201.1, U202.C2 (SRN), U204.2 (BAT), U204.3 (BAT)
- new net CC1: J202.A5 (CC1), R203.2
- new net CC2: J202.B5 (CC2), R204.2
- new net CHG: U204.9 (CHG)
- new net D+: U201.4 (I/O2)
- new net D-: U201.6 (I/O1)
- new net FT_3V3: Q201.1 (D)
- new net GAUGE_BIN: R202.1, U202.B1 (BIN)
- new net GAUGE_VDD: C201.1, U202.B3 (VDD)
- new net GND: C201.2, C202.2, C203.2, C204.2, C205.2, C206.2, C207.2, C208.2, C210.2, J201.1 (Pin_1), J202.A1 (GND), J202.A12 (GND), J202.B1 (GND), J202.B12 (GND), J202.SH (SHIELD), R202.2, R203.1, R204.1, R205.1, R206.1, R207.2, R209.2, U201.2 (GND), U202.B2 (VSS), U203.2 (GND), U204.15 (TD), U204.17 (VSS), U204.4 (CE), U204.5 (EN2), U204.6 (EN1), U204.8 (VSS), U205.2 (GND)
- new net GPOUT: U202.A1 (GPOUT)
- new net PGOOD: Q201.2 (G), R210.2, R211.2, U204.7 (PGOOD)
- new net SCL: U202.A3 (SCL)
- new net SDA: U202.A2 (SDA)
- new net USB_DM: J202.A7 (D-), J202.B7 (D-), U201.1 (I/O1)
- new net USB_DP: J202.A6 (D+), J202.B6 (D+), U201.3 (I/O2)
- new net USB_VBUS: F201.1, J202.A4 (VBUS), J202.A9 (VBUS), J202.B4 (VBUS), J202.B9 (VBUS)
- new net VBUS: C202.1, F201.2, U201.5 (VBUS), U204.13 (IN)
- new net VSYS: C203.1, C207.1, C208.1, L201.1, U203.1 (IN), U203.3 (EN), U204.10 (OUT), U204.11 (OUT), U205.4 (EN), U205.5 (VIN)
- no-connect marks 0 -> 3
Other:
- note added: "12V Rail"
- note added: "3V3 Rail"
- note added: "Battery"
- note added: "Battery Charger"
- note added: "Battery Gauge"
- note added: "Power Flags"
- note added: "Power Indicators and FT260 Power"
- note added: "USB C Power Configuration"
- note added: "USB Connector"

Commit message: fixed power side
Parts:
- added C211: 1u, Capacitor_SMD:C_0603_1608Metric, symbol Device:C
Connections:
- net GND: now also C211.2
- net VBUS: now also C211.1
- net D+ renamed USB_IN_D-
- net USB_IN_D-: now also J202.A6 (D+), J202.B6 (D+)
- net D- renamed USB_IN_D+
- net USB_IN_D+: now also J202.A7 (D-), J202.B7 (D-)
- removed net USB_DM: J202.A7 (D-), J202.B7 (D-), U201.1 (I/O1)
- removed net USB_DP: J202.A6 (D+), J202.B6 (D+), U201.3 (I/O2)
- new net USB_D+: U201.1 (I/O1)
- new net USB_D-: U201.3 (I/O2)

Commit message: Restarting routing
Parts:
- removed C201: 2.2u, Capacitor_SMD:C_0603_1608Metric, symbol Device:C
- removed C204: 1u, Capacitor_SMD:C_0603_1608Metric, symbol Device:C
- removed R201: 10m, Resistor_SMD:R_0603_1608Metric, symbol Device:R
- removed R202: 10k, Resistor_SMD:R_0603_1608Metric, symbol Device:R
- removed U202: BQ27426, Package_BGA:Texas_DSBGA-9_1.62x1.58mm_Layout3x3_P0.5mm, symbol picowy_symbols:BQ27426
- added C24: 0.47u, Capacitor_SMD:C_0603_1608Metric, symbol Device:C
- added C27: 1u, Capacitor_SMD:C_0603_1608Metric, symbol Device:C
- added R15: 10m, Resistor_SMD:R_0603_1608Metric, symbol Device:R
- added R16: 10k, Resistor_SMD:R_0603_1608Metric, symbol Device:R
- added U12: BQ27441-G1, Package_SON:Texas_S-PDSO-N12, symbol Battery_Management:BQ27441-G1
- BT1: renamed from BT201; now fitted
- J2: renamed from J201; symbol Connector_Generic:Conn_01x02 -> Connector_Generic:Conn_01x03
- U10: renamed from U204; footprint Package_DFN_QFN:VQFN-16-1EP_3x3mm_P0.5mm_EP1.68x1.68mm_ThermalVias -> Package_DFN_QFN:VQFN-16-1EP_3x3mm_P0.5mm_EP1.68x1.68mm
- renumbered C202 to C25, C203 to C26, C205 to C28, C211 to C29, C206 to C30, C207 to C31, C208 to C32, C209 to C33, C210 to C34, D201 to D1, F201 to F1, J202 to J3, L201 to L1, Q201 to Q1, R203 to R17, R204 to R18, R205 to R19, R206 to R20, R207 to R21, R208 to R22, R209 to R23, R210 to R24, R211 to R25, U205 to U11, U201 to U7, U203 to U9
Connections:
- net +BATT: now also J2.1 (Pin_1), C27.1, R15.2, U12.6 (BAT), U12.8 (SRP); no longer J2.2 (Pin_2)
- net BATT_IN: now also R15.1, U12.7 (SRN)
- net CHG: now also R24.2
- net GAUGE_BIN: now also R16.1, U12.10 (BIN)
- net GAUGE_VDD: now also C24.1, U12.5 (V_{DD})
- net GND: now also J2.3 (Pin_3), C24.2, C27.2, R16.2, U12.13 (PAD), U12.3 (V_{SS}); no longer J2.1 (Pin_1)
- net GPOUT: now also U12.12 (GPOUT)
- net PGOOD: no longer R24.2
- net SCL: now also U12.1 (SDA)
- net SDA: now also U12.2 (SCL)
- no-connect marks 3 -> 4
Other:
- note added: "*Decoupling Cap"
- note removed: "Power Flags"
- moved on the sheet: C26, C28, R17, R18, U9
