File: hardware/picowy.kicad_pcb (KiCad board)
At the start: 2 copper layers, 0 parts

Commit message: fixed power side
Parts:
- added C101: 100n, Capacitor_SMD:C_0603_1608Metric, F.Cu at (77.8, 63.0)
- added C102: 47p, Capacitor_SMD:C_0603_1608Metric, F.Cu at (124.0, 120.5)
- added C103: 47p, Capacitor_SMD:C_0603_1608Metric, F.Cu at (124.0, 117.3)
- added C104: 10u, Capacitor_SMD:C_0603_1608Metric, F.Cu at (77.8, 70.5)
- added C105: 100n, Capacitor_SMD:C_0603_1608Metric, F.Cu at (77.8, 73.0)
- added C106: 100n, Capacitor_SMD:C_0603_1608Metric, F.Cu at (77.8, 75.5)
- added C107: 4.7u, Capacitor_SMD:C_0603_1608Metric, F.Cu at (77.8, 78.0)
- added C108: 100n, Capacitor_SMD:C_0603_1608Metric, F.Cu at (77.8, 80.5)
- added C109: 100n, Capacitor_SMD:C_0603_1608Metric, F.Cu at (77.8, 83.0)
- added C110: 4.7u, Capacitor_SMD:C_0603_1608Metric, F.Cu at (77.8, 85.5)
- added C111: 4.7u, Capacitor_SMD:C_0603_1608Metric, F.Cu at (81.8, 63.0)
- added C112: 1u, Capacitor_SMD:C_0603_1608Metric, F.Cu at (81.8, 65.5)
- added C113: 100n, Capacitor_SMD:C_0603_1608Metric, F.Cu at (81.8, 68.0)
- added C114: 4.7u, Capacitor_SMD:C_0603_1608Metric, F.Cu at (81.8, 70.5)
- added C115: 4.7u, Capacitor_SMD:C_0603_1608Metric, F.Cu at (81.8, 73.0)
- added C116: 100n, Capacitor_SMD:C_0603_1608Metric, F.Cu at (81.8, 75.5)
- added C117: 100n, Capacitor_SMD:C_0603_1608Metric, F.Cu at (81.8, 78.0)
- added C118: 100n, Capacitor_SMD:C_0603_1608Metric, F.Cu at (81.8, 80.5)
- added C119: 10u, Capacitor_SMD:C_0603_1608Metric, F.Cu at (81.8, 83.0)
- added C120: 4.7u, Capacitor_SMD:C_0603_1608Metric, F.Cu at (81.8, 85.5)
- added C121: 1u, Capacitor_SMD:C_0603_1608Metric, F.Cu at (85.8, 63.0)
- added C122: 100n, Capacitor_SMD:C_0603_1608Metric, F.Cu at (85.8, 65.5)
- added C201: 2.2u, Capacitor_SMD:C_0603_1608Metric, F.Cu at (178.7, 98.1)
- added C202: 1u, Capacitor_SMD:C_0603_1608Metric, F.Cu at (149.2, 116.8)
- added C203: 1u, Capacitor_SMD:C_0603_1608Metric, F.Cu at (167.4, 96.0)
- added C204: 1u, Capacitor_SMD:C_0603_1608Metric, F.Cu at (175.7, 98.6)
- added C205: 1u, Capacitor_SMD:C_0603_1608Metric, F.Cu at (166.9, 101.8)
- added C206: 4.7u, Capacitor_SMD:C_0603_1608Metric, F.Cu at (171.1, 112.9)
- added C207: 10u, Capacitor_SMD:C_0603_1608Metric, F.Cu at (169.0, 80.1)
- added C208: 4.7u, Capacitor_SMD:C_0603_1608Metric, F.Cu at (170.2, 106.1)
- added C209: 4.7p, Capacitor_SMD:C_0603_1608Metric, F.Cu at (89.8, 63.0)
- added C210: 4.7u, Capacitor_SMD:C_0603_1608Metric, F.Cu at (89.8, 65.5)
- added C211: 1u, Capacitor_SMD:C_0603_1608Metric, F.Cu at (167.9, 107.4)
- added D201: STPS0530Z, Diode_SMD:D_SOD-123, F.Cu at (162.5, 80.3)
- added F201: VBUS Polyfuse, Fuse:Fuse_1206_3216Metric_Pad1.42x1.75mm_HandSolder, F.Cu at (151.0, 118.9)
- added J101: Conn_ARM_SWD_TagConnect_TC2030, Connector:Tag-Connect_TC2030-IDC-FP_2x03_P1.27mm_Vertical, F.Cu at (149.5, 95.3)
- added J201: Battery Connector, picowy_footprints:CONN_DF65-3P-1.7V21_HIR, F.Cu at (169.5, 87.8)
- added J202: USB_C_Receptacle_USB2.0_14P, picowy_footprints:CONN_124018612112A_AMP, F.Cu at (147.0, 121.9)
- added L201: 6.8u, Inductor_SMD:L_1210_3225Metric_Pad1.42x2.65mm_HandSolder, F.Cu at (166.0, 76.3)
- added NT101: OLED_GPIO_NT, NetTie:NetTie-2_SMD_Pad0.5mm, F.Cu at (114.9, 85.3)
- added Q201: PMOS, Package_TO_SOT_SMD:SOT-23-3, F.Cu at (154.7, 84.9)
- added R101: 5.1k, Resistor_SMD:R_0603_1608Metric, F.Cu at (115.7, 110.1)
- added R102: 1.4k, Resistor_SMD:R_0603_1608Metric, F.Cu at (89.8, 70.5)
- added R103: 1.4k, Resistor_SMD:R_0603_1608Metric, F.Cu at (89.8, 73.0)
- added R104: 33, Resistor_SMD:R_0603_1608Metric, F.Cu at (121.6, 119.8)
- added R105: 33, Resistor_SMD:R_0603_1608Metric, F.Cu at (121.6, 118.1)
- added R106: 1k, Resistor_SMD:R_0603_1608Metric, F.Cu at (89.8, 80.5)
- added R107: 1k, Resistor_SMD:R_0603_1608Metric, F.Cu at (89.8, 83.0)
- added R108: 910k, Capacitor_SMD:C_0603_1608Metric, F.Cu at (89.8, 85.5)
- added R109: 10k, Resistor_SMD:R_0603_1608Metric, F.Cu at (93.8, 63.0)
- added R110: 10k, Resistor_SMD:R_0603_1608Metric, F.Cu at (93.8, 65.5)
- added R111: 10k, Resistor_SMD:R_0603_1608Metric, F.Cu at (93.8, 68.0)
- added R112: 10k, Resistor_SMD:R_0603_1608Metric, F.Cu at (93.8, 70.5)
- added R113: 4.7k, Resistor_SMD:R_0603_1608Metric, F.Cu at (93.8, 73.0)
- added R114: 10k, Resistor_SMD:R_0603_1608Metric, F.Cu at (93.8, 75.5)
- added R115: 2.2k, Resistor_SMD:R_0603_1608Metric, F.Cu at (93.8, 78.0)
- added R116: 2.2k, Resistor_SMD:R_0603_1608Metric, F.Cu at (93.8, 80.5)
- added R201: 10m, Resistor_SMD:R_0603_1608Metric, F.Cu at (172.2, 97.6)
- added R202: 10k, Resistor_SMD:R_0603_1608Metric, F.Cu at (178.4, 100.4)
- added R203: 5.1k, Resistor_SMD:R_0603_1608Metric, F.Cu at (143.8, 124.1)
- added R204: 5.1k, Resistor_SMD:R_0603_1608Metric, F.Cu at (156.3, 124.9)
- added R205: 17.4k, Resistor_SMD:R_0603_1608Metric, F.Cu at (166.8, 111.5)
- added R206: 30k, Resistor_SMD:R_0603_1608Metric, F.Cu at (166.8, 109.8)
- added R207: 10k, Resistor_SMD:R_0603_1608Metric, F.Cu at (169.5, 112.9)
- added R208: 1.8M, Resistor_SMD:R_0603_1608Metric, F.Cu at (97.8, 75.5)
- added R209: 205k, Resistor_SMD:R_0603_1608Metric, F.Cu at (97.8, 78.0)
- added R210: 10k, Resistor_SMD:R_0603_1608Metric, F.Cu at (97.8, 80.5)
- added R211: 10k, Resistor_SMD:R_0603_1608Metric, F.Cu at (97.8, 83.0)
- added U101: ER-TP1.44-1, picowy_footprints:ER-TP1.44-1, F.Cu at (140.3, 74.2)
- added U102: LIS2HH12, Package_LGA:LGA-12_2x2mm_P0.5mm, F.Cu at (129.2, 79.2)
- added U103: FT260Q, Package_DFN_QFN:WQFN-28-1EP_4x4mm_P0.4mm_EP2.7x2.7mm, F.Cu at (131.3, 111.2)
- added U104: ER-OLED1.12-2W, picowy_footprints:ER-CON20HT-1, F.Cu at (150.0, 71.6)
- added U105: AT24CS04-SSHM, Package_SO:SOIC-8_3.9x4.9mm_P1.27mm, F.Cu at (126.0, 100.0)
- added U106: STM32L011G4Ux, Package_DFN_QFN:QFN-28_4x4mm_P0.5mm, F.Cu at (132.5, 88.0)
- added U201: USBLC6-2SC6, Package_TO_SOT_SMD:SOT-23-6, F.Cu at (145.1, 118.3)
- added U202: BQ27426, Package_BGA:Texas_DSBGA-9_1.62x1.58mm_Layout3x3_P0.5mm, F.Cu at (174.9, 101.4)
- added U203: TPS7A20xxxDBV, Package_TO_SOT_SMD:SOT-23-5, F.Cu at (167.3, 98.8)
- added U204: BQ24230RGT, Package_DFN_QFN:VQFN-16-1EP_3x3mm_P0.5mm_EP1.68x1.68mm_ThermalVias, F.Cu at (170.8, 109.0)
- added U205: TPS61040DDC, Package_TO_SOT_SMD:SOT-23-5, F.Cu at (166.0, 80.2)
Other:
- board outline added: 56 x 66 mm
- copper layers 2 -> 4

Commit message: Restarting routing
Parts:
- removed C101, C105, C106, C108, C109, C113, C116, C117, C118, C122: 100n, Capacitor_SMD:C_0603_1608Metric
- removed C102, C103: 47p, Capacitor_SMD:C_0603_1608Metric
- removed C104, C119, C207: 10u, Capacitor_SMD:C_0603_1608Metric
- removed C107, C110, C111, C114, C115, C120, C206, C208, C210: 4.7u, Capacitor_SMD:C_0603_1608Metric
- removed C112, C121, C202, C203, C204, C205, C211: 1u, Capacitor_SMD:C_0603_1608Metric
- removed C201: 2.2u, Capacitor_SMD:C_0603_1608Metric
- removed C209: 4.7p, Capacitor_SMD:C_0603_1608Metric
- removed D201: STPS0530Z, Diode_SMD:D_SOD-123
- removed F201: VBUS Polyfuse, Fuse:Fuse_1206_3216Metric_Pad1.42x1.75mm_HandSolder
- removed J101: Conn_ARM_SWD_TagConnect_TC2030, Connector:Tag-Connect_TC2030-IDC-FP_2x03_P1.27mm_Vertical
- removed J201: Battery Connector, picowy_footprints:CONN_DF65-3P-1.7V21_HIR
- removed J202: USB_C_Receptacle_USB2.0_14P, picowy_footprints:CONN_124018612112A_AMP
- removed L201: 6.8u, Inductor_SMD:L_1210_3225Metric_Pad1.42x2.65mm_HandSolder
- removed NT101: OLED_GPIO_NT, NetTie:NetTie-2_SMD_Pad0.5mm
- removed Q201: PMOS, Package_TO_SOT_SMD:SOT-23-3
- removed R101, R203, R204: 5.1k, Resistor_SMD:R_0603_1608Metric
- removed R102, R103: 1.4k, Resistor_SMD:R_0603_1608Metric
- removed R104, R105: 33, Resistor_SMD:R_0603_1608Metric
- removed R106, R107: 1k, Resistor_SMD:R_0603_1608Metric
- removed R108: 910k, Capacitor_SMD:C_0603_1608Metric
- removed R109, R110, R111, R112, R114, R202, R207, R210, R211: 10k, Resistor_SMD:R_0603_1608Metric
- removed R113: 4.7k, Resistor_SMD:R_0603_1608Metric
- removed R115, R116: 2.2k, Resistor_SMD:R_0603_1608Metric
- removed R201: 10m, Resistor_SMD:R_0603_1608Metric
- removed R205: 17.4k, Resistor_SMD:R_0603_1608Metric
- removed R206: 30k, Resistor_SMD:R_0603_1608Metric
- removed R208: 1.8M, Resistor_SMD:R_0603_1608Metric
- removed R209: 205k, Resistor_SMD:R_0603_1608Metric
- removed U101: ER-TP1.44-1, picowy_footprints:ER-TP1.44-1
- removed U102: LIS2HH12, Package_LGA:LGA-12_2x2mm_P0.5mm
- removed U103: FT260Q, Package_DFN_QFN:WQFN-28-1EP_4x4mm_P0.4mm_EP2.7x2.7mm
- removed U104: ER-OLED1.12-2W, picowy_footprints:ER-CON20HT-1
- removed U105: AT24CS04-SSHM, Package_SO:SOIC-8_3.9x4.9mm_P1.27mm
- removed U106: STM32L011G4Ux, Package_DFN_QFN:QFN-28_4x4mm_P0.5mm
- removed U201: USBLC6-2SC6, Package_TO_SOT_SMD:SOT-23-6
- removed U202: BQ27426, Package_BGA:Texas_DSBGA-9_1.62x1.58mm_Layout3x3_P0.5mm
- removed U203: TPS7A20xxxDBV, Package_TO_SOT_SMD:SOT-23-5
- removed U204: BQ24230RGT, Package_DFN_QFN:VQFN-16-1EP_3x3mm_P0.5mm_EP1.68x1.68mm_ThermalVias
- removed U205: TPS61040DDC, Package_TO_SOT_SMD:SOT-23-5
- added C1: 100n, Capacitor_SMD:C_0603_1608Metric, F.Cu at (85.5, 36.8)
- added C10: 1u, Capacitor_SMD:C_0603_1608Metric, F.Cu at (85.5, 59.3)
- added C11: 100n, Capacitor_SMD:C_0603_1608Metric, F.Cu at (85.5, 61.9)
- added C12: 100n, Capacitor_SMD:C_0603_1608Metric, F.Cu at (89.5, 36.8)
- added C13: 100n, Capacitor_SMD:C_0603_1608Metric, F.Cu at (89.5, 39.3)
- added C14: 4.7u, Capacitor_SMD:C_0603_1608Metric, F.Cu at (89.5, 41.8)
- added C15: 4.7u, Capacitor_SMD:C_0603_1608Metric, F.Cu at (89.5, 44.3)
- added C16: 1u, Capacitor_SMD:C_0603_1608Metric, F.Cu at (89.5, 46.8)
- added C17: 4.7u, Capacitor_SMD:C_0603_1608Metric, F.Cu at (89.5, 49.3)
- added C18: 100n, Capacitor_SMD:C_0603_1608Metric, F.Cu at (89.5, 51.8)
- added C19: 100n, Capacitor_SMD:C_0603_1608Metric, F.Cu at (89.5, 54.3)
- added C2: 47p, Capacitor_SMD:C_0603_1608Metric, F.Cu at (85.5, 39.3)
- added C20: 100n, Capacitor_SMD:C_0603_1608Metric, F.Cu at (89.5, 56.8)
- added C21: 10u, Capacitor_SMD:C_0603_1608Metric, F.Cu at (89.5, 59.3)
- added C22: 1u, Capacitor_SMD:C_0603_1608Metric, F.Cu at (89.5, 61.9)
- added C23: 100n, Capacitor_SMD:C_0603_1608Metric, F.Cu at (93.5, 36.8)
- added C24: 0.47u, Capacitor_SMD:C_0603_1608Metric, F.Cu at (93.5, 39.3)
- added C25: 1u, Capacitor_SMD:C_0603_1608Metric, F.Cu at (93.5, 41.8)
- added C26: 1u, Capacitor_SMD:C_0603_1608Metric, F.Cu at (93.5, 44.3)
- added C27: 1u, Capacitor_SMD:C_0603_1608Metric, F.Cu at (93.5, 46.8)
- added C28: 1u, Capacitor_SMD:C_0603_1608Metric, F.Cu at (93.5, 49.3)
- added C29: 1u, Capacitor_SMD:C_0603_1608Metric, F.Cu at (93.5, 51.8)
- added C3: 47p, Capacitor_SMD:C_0603_1608Metric, F.Cu at (85.5, 41.8)
- added C30: 4.7u, Capacitor_SMD:C_0603_1608Metric, F.Cu at (93.5, 54.3)
- added C31: 10u, Capacitor_SMD:C_0603_1608Metric, F.Cu at (93.5, 56.8)
- added C32: 4.7u, Capacitor_SMD:C_0603_1608Metric, F.Cu at (93.5, 59.3)
- added C33: 4.7p, Capacitor_SMD:C_0603_1608Metric, F.Cu at (93.5, 61.9)
- added C34: 4.7u, Capacitor_SMD:C_0603_1608Metric, F.Cu at (97.5, 36.8)
- added C4: 10u, Capacitor_SMD:C_0603_1608Metric, F.Cu at (85.5, 44.3)
- added C5: 100n, Capacitor_SMD:C_0603_1608Metric, F.Cu at (85.5, 46.8)
- added C6: 100n, Capacitor_SMD:C_0603_1608Metric, F.Cu at (85.5, 49.3)
- added C7: 4.7u, Capacitor_SMD:C_0603_1608Metric, F.Cu at (85.5, 51.8)
- added C8: 4.7u, Capacitor_SMD:C_0603_1608Metric, F.Cu at (85.5, 54.3)
- added C9: 4.7u, Capacitor_SMD:C_0603_1608Metric, F.Cu at (85.5, 56.8)
- added D1: STPS0530Z, Diode_SMD:D_SOD-123, F.Cu at (104.3, 72.3)
- added F1: VBUS Polyfuse, Fuse:Fuse_1206_3216Metric_Pad1.42x1.75mm_HandSolder, F.Cu at (104.4, 69.0)
- added J1: Conn_ARM_SWD_TagConnect_TC2030, Connector:Tag-Connect_TC2030-IDC-FP_2x03_P1.27mm_Vertical, F.Cu at (112.3, 56.5)
- added J2: Battery Connector, picowy_footprints:CONN_DF65-3P-1.7V21_HIR, F.Cu at (113.4, 47.9)
- added J3: USB_C_Receptacle_USB2.0_14P, picowy_footprints:CONN_124018612112A_AMP, F.Cu at (90.4, 69.4)
- added L1: 6.8u, Inductor_SMD:L_1210_3225Metric_Pad1.42x2.65mm_HandSolder, F.Cu at (99.2, 65.2)
- added NT1: OLED_GPIO_NT, NetTie:NetTie-2_SMD_Pad0.5mm, F.Cu at (120.6, 68.6)
- added NT2: FT_GPIO_GND, NetTie:NetTie-2_SMD_Pad0.5mm, F.Cu at (120.6, 70.1)
- added Q1: PMOS, Package_TO_SOT_SMD:SOT-23-3, F.Cu at (98.8, 69.5)
- added R1: 5.1k, Resistor_SMD:R_0603_1608Metric, F.Cu at (97.5, 39.3)
- added R10: 4.7k, Resistor_SMD:R_0603_1608Metric, F.Cu at (97.5, 61.9)
- added R11: 2.2k, Resistor_SMD:R_0603_1608Metric, F.Cu at (101.5, 36.8)
- added R12: 2.2k, Resistor_SMD:R_0603_1608Metric, F.Cu at (101.5, 39.3)
- added R13: 10k, Resistor_SMD:R_0603_1608Metric, F.Cu at (101.5, 41.8)
- added R14: 10k, Resistor_SMD:R_0603_1608Metric, F.Cu at (101.5, 44.3)
- added R15: 10m, Resistor_SMD:R_0603_1608Metric, F.Cu at (101.5, 46.8)
- added R16: 10k, Resistor_SMD:R_0603_1608Metric, F.Cu at (101.5, 49.3)
- added R17: 5.1k, Resistor_SMD:R_0603_1608Metric, F.Cu at (101.5, 51.8)
- added R18: 5.1k, Resistor_SMD:R_0603_1608Metric, F.Cu at (101.5, 54.3)
- added R19: 17.4k, Resistor_SMD:R_0603_1608Metric, F.Cu at (101.5, 56.8)
- added R2: 1.4k, Resistor_SMD:R_0603_1608Metric, F.Cu at (97.5, 41.8)
- added R20: 30k, Resistor_SMD:R_0603_1608Metric, F.Cu at (101.5, 59.3)
- added R21: 10k, Resistor_SMD:R_0603_1608Metric, F.Cu at (101.5, 61.9)
- added R22: 1.8M, Resistor_SMD:R_0603_1608Metric, F.Cu at (105.6, 36.8)
- added R23: 205k, Resistor_SMD:R_0603_1608Metric, F.Cu at (105.6, 39.3)
- added R24: 10k, Resistor_SMD:R_0603_1608Metric, F.Cu at (105.6, 41.8)
- added R25: 10k, Resistor_SMD:R_0603_1608Metric, F.Cu at (105.6, 44.3)
- added R26: 10k, Resistor_SMD:R_0603_1608Metric, F.Cu at (105.6, 46.8)
- added R3: 1.4k, Resistor_SMD:R_0603_1608Metric, F.Cu at (97.5, 44.3)
- added R4: 33, Resistor_SMD:R_0603_1608Metric, F.Cu at (97.5, 46.8)
- added R5: 33, Resistor_SMD:R_0603_1608Metric, F.Cu at (97.5, 49.3)
- added R6: 1k, Resistor_SMD:R_0603_1608Metric, F.Cu at (97.5, 51.8)
- added R7: 1k, Resistor_SMD:R_0603_1608Metric, F.Cu at (97.5, 54.3)
- added R8: 10k, Resistor_SMD:R_0603_1608Metric, F.Cu at (97.5, 56.8)
- added R9: 910k, Capacitor_SMD:C_0603_1608Metric, F.Cu at (97.5, 59.3)
- added U1: ER-TP1.44-1, picowy_footprints:ER-TP1.44-1, F.Cu at (98.6, 73.0)
- added U10: BQ24230RGT, Package_DFN_QFN:VQFN-16-1EP_3x3mm_P0.5mm_EP1.68x1.68mm, F.Cu at (121.0, 44.5)
- added U11: TPS61040DDC, Package_TO_SOT_SMD:SOT-23-5, F.Cu at (110.1, 72.9)
- added U12: BQ27441-G1, Package_SON:Texas_S-PDSO-N12, F.Cu at (121.0, 49.4)
- added U2: LIS2HH12, Package_LGA:LGA-12_2x2mm_P0.5mm, F.Cu at (104.2, 65.1)
- added U3: FT260Q, picowy_footprints:WQFN-28_FTD, F.Cu at (120.2, 55.3)
- added U4: ER-OLED1.12-2W, picowy_footprints:ER-CON20HT-1, F.Cu at (166.4, 100.2)
- added U5: AT24CS04-SSHM, Package_SO:SOIC-8_3.9x4.9mm_P1.27mm, F.Cu at (116.9, 64.6)
- added U6: STM32L011G4Ux, Package_DFN_QFN:QFN-28_4x4mm_P0.5mm, F.Cu at (116.2, 71.0)
- added U7: USBLC6-2SC6, Package_TO_SOT_SMD:SOT-23-6, F.Cu at (110.1, 63.7)
- added U9: TPS7A20xxxDBV, Package_TO_SOT_SMD:SOT-23-5, F.Cu at (110.1, 68.3)
Routing:
- added copper zone on In1.Cu, net GND
- added copper zone on In2.Cu, net GND
Other:
- outline, holes or cut-outs redrawn
- rule solder_mask_min_width: 0.1 -> 0.15
- board text added: "DISPLAY"
- board text added: "TOUCH PANEL"

Commit message: Finished Board for Fabrication
Parts:
- added G***: Back_Pattern, picowy_footprints:Back_Pattern, F.Cu at (150.0, 94.8)
- added NT3: OLED_GPIO_NT2, NetTie:NetTie-2_SMD_Pad0.5mm, F.Cu at (164.8, 100.0)
- J3: footprint picowy_footprints:CONN_124018612112A_AMP -> picowy_footprints:2130830005_MOL
- moved C25 105.1 mm to (159.0, 124.0), turned to 90 degrees
- moved C13 100.9 mm to (164.5, 106.8), turned to -90 degrees
- moved C2 98.4 mm to (138.0, 122.5), turned to -90 degrees
- moved C14 98.1 mm to (163.0, 106.8), turned to -90 degrees
- moved C34 98.0 mm to (163.8, 109.0), turned to 180 degrees
- moved C1 97.4 mm to (162.0, 97.0), turned to 180 degrees
- moved C15 95.6 mm to (163.8, 104.5), turned to 180 degrees
- moved R23 95.4 mm to (164.5, 114.2), turned to -90 degrees
- moved R22 95.0 mm to (164.5, 111.2), turned to -90 degrees
- moved C31 94.7 mm to (167.2, 116.2), turned to 180 degrees
- moved C3 93.0 mm to (138.0, 118.5), turned to 90 degrees
- moved C4 92.1 mm to (162.0, 95.5), turned to 180 degrees
- moved C6 90.2 mm to (164.3, 93.2), turned to 90 degrees
- moved C10 89.6 mm to (163.8, 103.0), turned to 180 degrees
- moved C23 86.6 mm to (165.5, 85.0), turned to 180 degrees
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Connections:
- net /Main System/FT_SCL renamed /Main System/FT.SCL
- net /Main System/FT_SDA renamed /Main System/FT.SDA
- net MCU_RX renamed MCU.RX
- net MCU_TX renamed MCU.TX
- net MISO renamed MCU.MISO
- net MOSI renamed MCU.MOSI
- net Net-(U10-ISET) renamed /Power System/CHG_ISET
- net Net-(U10-TMR) renamed /Power System/CHG_TMR
- net Net-(U10-TS) renamed /Power System/CHG_TS
- net SCLK renamed MCU.SCLK
- net SWCLK renamed MCU.SWCLK
- net SWDIO renamed MCU.SWDIO
- C31 pad 1: VSYS -> +3V3
- J3 pad A8: (no net) -> unconnected-(J3-SBU1-PadA8)
- J3 pad B8: (no net) -> unconnected-(J3-SBU2-PadB8)
- L1 pad 1: VSYS -> +3V3
- R11 pad 2: SDA -> MCU.SDA
- R12 pad 1: +3V3 -> MCU.SCL
- R12 pad 2: SCL -> +3V3
- U11 pad 4: VSYS -> +3V3
- U11 pad 5: VSYS -> +3V3
- U12 pad 1: SCL -> MCU.SDA
- U12 pad 2: SDA -> MCU.SCL
- U4 pad 10: /Main System/OLED_GPIO_GND -> /Main System/OLED_GPIO_GND2
- U4 pad 11: /Main System/OLED_GPIO_GND -> /Main System/OLED_GPIO_GND2
- U6 pad 10: unconnected-(U6-PA4-Pad10) -> ~{CS_ACCEL}
- U6 pad 14: PGOOD -> DC_OLED
- U6 pad 15: CHG -> ~{RES_OLED}
- U6 pad 18: GPOUT -> ~{CS_OLED}
- U6 pad 23: ~{CS_ACCEL} -> unconnected-(U6-PA15-Pad23)
- U6 pad 24: DC_OLED -> CHG
- U6 pad 25: ~{RES_OLED} -> PGOOD
- U6 pad 26: ~{CS_OLED} -> GPOUT
- U6 pad 27: SCL -> MCU.SCL
- U6 pad 28: SDA -> MCU.SDA
- U6 pad 6: YD -> XR
- U6 pad 7: XL -> YD
- U6 pad 9: XR -> XL
Routing:
- net GND: track 0.00 -> 121.2 mm, vias 0 -> 66
- net NRST: track 0.00 -> 92.1 mm, vias 0 -> 3
- net PGOOD: track 0.00 -> 71.8 mm, vias 0 -> 2
- net MCU.TX: track 0.00 -> 71.3 mm, vias 0 -> 2
- net MCU.RX: track 0.00 -> 67.3 mm, vias 0 -> 2
- net BOOT0: track 0.00 -> 60.0 mm, vias 0 -> 2
- net +3V3: track 0.00 -> 55.3 mm, vias 0 -> 25
- net FT_3V3: track 0.00 -> 48.0 mm, vias 0 -> 13
- net ~{CS_OLED}: track 0.00 -> 46.6 mm
- net MCU.SCLK: track 0.00 -> 38.2 mm
- net MCU.MOSI: track 0.00 -> 38.2 mm, vias 0 -> 3
- net ~{RES_OLED}: track 0.00 -> 32.9 mm
- net CHG: track 0.00 -> 32.7 mm
- net DC_OLED: track 0.00 -> 29.6 mm
- net VBUS: track 0.00 -> 29.3 mm, vias 0 -> 5
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- added copper zone on B.Cu, net +3V3
- added copper zone on F.Cu, net +3V3
- added copper zone on F.Cu, net +BATT
- added copper zone on F.Cu, net /Power System/USB_VBUS
- added copper zone on F.Cu, net BATT_IN
- added copper zone on B.Cu, net FT_3V3
- added copper zone on F.Cu, net FT_3V3
- added copper zone on B.Cu, net VBUS
Other:
- board size 56 x 66 mm -> 56 x 65.5 mm
- board text added: "+3V3"
- board text added: "BATTERY"
- board text added: "CUTOUT"
- board text added: "FROM: WYATT"
- board text added: "FT_3V3"
- board text added: "GND"
- board text added: "TO: <3 <3 <3 GAHYEON"
