File: hardware/picowy.kicad_sch (KiCad schematic)
At the start: 0 parts

Commit message: Added accelerometer schematic
Parts:
- added C1: 10u, Capacitor_SMD:C_0603_1608Metric, symbol Device:C
- added C2, C3: 100n, Capacitor_SMD:C_0603_1608Metric, symbol Device:C
- added U1: LIS2HH12, Package_LGA:LGA-12_2x2mm_P0.5mm, symbol Sensor_Motion:LIS2HH12
Connections:
- new net +3V3: C1.1, C2.1, C3.1, U1.10 (Vdd_IO), U1.9 (Vdd)
- new net GND: C1.2, C2.2, C3.2, U1.5 (RES), U1.6 (GND), U1.7 (GND), U1.8 (GND)
- new net MISO: U1.3 (SA0/SDO)
- new net MOSI: U1.4 (SDA/SDI)
- new net SCLK: U1.1 (SCL/SPC)
- new net ~{CS_ACCEL}: U1.2 (~{CS})
- no-connect marks 0 -> 2
Other:
- note added: "Accelerometer"
- company: (none) -> eklipsed
- title: (none) -> Main System

Commit message: finished schematic
Parts:
- added C102, C103: 47p, Capacitor_SMD:C_0603_1608Metric, symbol Device:C
- added C105, C108, C109, C113, C116, C117, C118, C122: 100n, Capacitor_SMD:C_0603_1608Metric, symbol Device:C
- added C107, C110, C111, C114, C115, C120: 4.7u, Capacitor_SMD:C_0603_1608Metric, symbol Device:C
- added C112, C121: 1u, Capacitor_SMD:C_0603_1608Metric, symbol Device:C
- added C119: 10u, Capacitor_SMD:C_0603_1608Metric, symbol Device:C
- added J101: Conn_ARM_SWD_TagConnect_TC2030, Connector:Tag-Connect_TC2030-IDC-FP_2x03_P1.27mm_Vertical, symbol Connector:Conn_ARM_SWD_TagConnect_TC2030
- added NT101: OLED_GPIO_NT, NetTie:NetTie-2_SMD_Pad0.5mm, symbol Device:NetTie_2
- added R101: 5.1k, Resistor_SMD:R_0603_1608Metric, symbol Device:R
- added R102, R103: 1.4k, Resistor_SMD:R_0603_1608Metric, symbol Device:R
- added R104, R105: 33, Resistor_SMD:R_0603_1608Metric, symbol Device:R
- added R106, R107: 1k, Resistor_SMD:R_0603_1608Metric, symbol Device:R
- added R108: 910k, Capacitor_SMD:C_0603_1608Metric, symbol Device:R
- added R109, R110, R111, R112, R114: 10k, Resistor_SMD:R_0603_1608Metric, symbol Device:R
- added R113: 4.7k, Resistor_SMD:R_0603_1608Metric, symbol Device:R
- added R115, R116: 2.2k, Resistor_SMD:R_0603_1608Metric, symbol Device:R
- added U101: ER-TP1.44-1, picowy_footprints:ER-TP1.44-1, symbol picowy_symbols:ER-TP1.44-1
- added U103: FT260Q, Package_DFN_QFN:WQFN-28-1EP_4x4mm_P0.4mm_EP2.7x2.7mm, symbol picowy_symbols:FT260Q
- added U104: ER-OLED1.12-2W, picowy_footprints:ER-CON20HT-1, symbol picowy_symbols:ER-OLED1.12-2W
- added U105: AT24CS04-SSHM, Package_SO:SOIC-8_3.9x4.9mm_P1.27mm, symbol Memory_EEPROM:AT24CS04-SSHM
- added U106: STM32L011G4Ux, Package_DFN_QFN:QFN-28_4x4mm_P0.5mm, symbol MCU_ST_STM32L0:STM32L011G4Ux
- renumbered C2 to C101, C1 to C104, C3 to C106, U1 to U102
Connections:
- net +3V3: now also C112.1, C116.1, C119.1, C121.1, C122.1, J101.1 (VCC), R114.1, R115.1, R116.1, U104.3 (VDD), U106.17 (VDD), U106.5 (VDDA)
- net GND: now also C102.2, C103.2, C105.2, C107.2, C108.2, C109.2, C110.2, C111.2, C112.2, C113.2, C114.2, C115.2, C116.2, C117.2, C118.2, C119.2, C120.2, C121.2, C122.2, J101.5 (GND), NT101.1, R108.2, R111.2, U103.19 (GND), U103.24 (AGND), U103.4 (DCNF0), U104.20 (GND), U104.4 (BS1), U104.5 (BS2), U105.2 (A1), U105.3 (A2), U105.4 (GND), U105.7 (WP), U106.16 (VSS)
- net MISO: now also U106.12 (PA6)
- net MOSI: now also U104.13 (D1/MOSI), U106.13 (PA7)
- net SCLK: now also U104.12 (D0/SCLK), U106.11 (PA5)
- net ~{CS_ACCEL}: now also U106.26 (PB5)
- new net +12V: C113.1, C114.1, U104.1 (VPP)
- new net BOOT0: C118.1, R111.1, U103.15 (DIO8), U106.1 (PB9)
- new net CHG: U106.14 (PB0)
- new net D+: C103.1, R105.2
- new net D-: C102.1, R104.1
- new net DC_OLED: U104.9 (A0/DC), U106.10 (PA4)
- new net DM: R104.2, U103.20 (DM)
- new net DP: R105.1, U103.21 (DP)
- new net FT_3V3: C105.1, C107.1, C108.1, C109.1, C110.1, C111.1, R106.1, R107.1, R109.1, R110.1, R112.1, R113.1, U103.22 (VOUT3V3), U103.23 (VCCIN), U103.6 (VCCIO), U105.8 (VCC)
- new net FT_DBG_DBGR: R109.2, U103.1 (DEBUGGER)
- new net FT_DBG_RSTN: R110.2, U103.2 (STEST_RSTN)
- new net FT_DCNF1: R112.2, U103.5 (DCNF1)
- new net FT_RESETN: C120.1, R113.2, U103.3 (RESETN)
- new net FT_SCL: R107.2, U103.13 (DIO6), U105.6 (SCL)
- new net FT_SDA: R106.2, U103.12 (DIO5), U105.5 (SDA)
- new net FT_VBUS_DET: R101.1, U103.26 (VBUS_DET)
- new net GPOUT: R114.2, U106.18 (PA8)
- new net IREF: R108.1, U104.6 (IREF)
- new net MCU_RX: U103.11 (DIO4), U106.28 (PB7)
- new net MCU_TX: U103.10 (DIO3), U106.27 (PB6)
- new net NRST: C117.1, J101.3 (~{RESET}), U103.14 (DIO7), U106.4 (NRST)
- new net OLED_GPIO_GND: NT101.2, U104.10 (~{WR}), U104.11 (E/~{RD}), U104.15 (D3), U104.16 (D4), U104.17 (D5), U104.18 (D6), U104.19 (D7)
- new net PGOOD: U106.15 (PB1)
- new net SCL: R115.2, U106.19 (PA9)
- new net SDA: R116.2, U106.20 (PA10)
- new net SWCLK: J101.4 (SWCLK), U106.22 (PA14)
- new net SWDIO: J101.2 (SWDIO), U106.21 (PA13)
- new net VBUS: R101.2
- new net VCOMH: C115.1, U104.2 (VCOMH)
- new net XL: U101.XL (1), U106.6 (PA0)
- new net XR: R103.2, U106.8 (PA2)
- new net XR_TP: R103.1, U101.XR (3)
- new net YD: R102.2, U106.9 (PA3)
- new net YD_TP: R102.1, U101.YD (2)
- new net YU: U101.YU (4), U106.7 (PA1)
- new net ~{CS_OLED}: U104.7 (~{CS}), U106.25 (PB4)
- new net ~{RES_OLED}: U104.8 (~{RES}), U106.24 (PB3)
- no-connect marks 2 -> 16
Other:
- note added: "*Filtering caps place next to connector after ESD protection"
- note added: "Configuration EEPROM"
- note added: "Debug Connector"
- note added: "FT260 Configuration"
- note added: "FTDI Firmware Flasher"
- note added: "Microcontroller"
- note added: "OLED Display"
- note added: "Touch Panel"
- moved on the sheet: C101, C104, C106, U102

Commit message: fixed power side
Parts:
- removed C108, C109: 100n, Capacitor_SMD:C_0603_1608Metric, symbol Device:C
- removed C110, C111: 4.7u, Capacitor_SMD:C_0603_1608Metric, symbol Device:C
Connections:
- net D+ renamed USB_D+
- net D- renamed USB_D-
- net DM renamed FT_D-
- net DP renamed FT_D+
Other:
- moved on the sheet: C105, C107, R104, R105

Commit message: Restarting routing
Parts:
- removed R110, R112, R114: 10k, Resistor_SMD:R_0603_1608Metric, symbol Device:R
- removed R115, R116: 2.2k, Resistor_SMD:R_0603_1608Metric, symbol Device:R
- added C11, C12: 100n, Capacitor_SMD:C_0603_1608Metric, symbol Device:C
- added C16: 1u, Capacitor_SMD:C_0603_1608Metric, symbol Device:C
- added C8, C9: 4.7u, Capacitor_SMD:C_0603_1608Metric, symbol Device:C
- added NT2: FT_GPIO_GND, NetTie:NetTie-2_SMD_Pad0.5mm, symbol Device:NetTie_2
- added R11, R12: 2.2k, Resistor_SMD:R_0603_1608Metric, symbol Device:R
- added R14, R26: 10k, Resistor_SMD:R_0603_1608Metric, symbol Device:R
- U3: renamed from U103; footprint Package_DFN_QFN:WQFN-28-1EP_4x4mm_P0.4mm_EP2.7x2.7mm -> picowy_footprints:WQFN-28_FTD; Manufacturer PN FT260Q-T -> FT260S-U
- renumbered C101 to C1, C112 to C10, C113 to C13, C114 to C14, C115 to C15, C120 to C17, C116 to C18, C117 to C19, C102 to C2, C118 to C20, C119 to C21, C121 to C22, C122 to C23, C103 to C3, C104 to C4, C105 to C5, C106 to C6, C107 to C7, J101 to J1, NT101 to NT1, R101 to R1, R113 to R10, R111 to R13, R102 to R2, R103 to R3, R104 to R4, R105 to R5, R106 to R6, R107 to R7, R109 to R8, R108 to R9, U101 to U1, U102 to U2, U104 to U4, U105 to U5, U106 to U6
Connections:
- net FT_DBG_RSTN is gone; now on net FT_GPIO_HI: U3.2 (STEST_RSTN)
- net +3V3: now also R11.1, R12.1, R14.1
- net BOOT0: now also U3.8 (DIO1); no longer U3.15 (DIO8)
- net CHG: now also U6.15 (PB1); no longer U6.14 (PB0)
- net DC_OLED: now also U6.24 (PB3); no longer U6.10 (PA4)
- net FT_3V3: now also C11.1, C12.1, C16.1, C8.1, C9.1, R26.1
- net FT_DCNF1: now also R26.2
- net GND: now also C11.2, C12.2, C16.2, C8.2, C9.2, NT2.1; no longer U3.4 (DCNF0)
- net GPOUT: now also R14.2
- net MCU_RX: now also U6.20 (PA10); no longer U6.28 (PB7)
- net MCU_TX: now also U6.19 (PA9); no longer U6.27 (PB6)
- net NRST: now also U3.7 (DIO0); no longer U3.14 (DIO7)
- net PGOOD: now also U6.14 (PB0); no longer U6.15 (PB1)
- net SCL: now also U6.27 (PB6), R12.2; no longer U6.19 (PA9)
- net SDA: now also U6.28 (PB7), R11.2; no longer U6.20 (PA10)
- net XL: now also U1.1 (XL), U6.7 (PA1); no longer U1.XL (1), U6.6 (PA0)
- net XR: now also U6.9 (PA3); no longer U6.8 (PA2)
- net XR_TP: now also U1.3 (XR); no longer U1.XR (3)
- net YD: now also U6.6 (PA0); no longer U6.9 (PA3)
- net YD_TP: now also U1.2 (YD); no longer U1.YD (2)
- net YU: now also U1.4 (YU), U6.8 (PA2); no longer U1.YU (4), U6.7 (PA1)
- net ~{CS_ACCEL}: now also U6.23 (PA15); no longer U6.26 (PB5)
- net ~{CS_OLED}: now also U6.26 (PB5); no longer U6.25 (PB4)
- net ~{RES_OLED}: now also U6.25 (PB4); no longer U6.24 (PB3)
- net FT_DBG_DBGR renamed FT_GPIO_HI
- new net FT_GPIO_LO: NT2.2, U3.4 (DCNF0)
Other:
- moved on the sheet: C10, C13, C14, C15, C17, C18, C19, C20, C21, C22, C23, J1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

Commit message: Finished Board for Fabrication
Parts:
- added NT3: OLED_GPIO_NT2, NetTie:NetTie-2_SMD_Pad0.5mm, symbol Device:NetTie_2
Connections:
- net +3V3: now also R12.2; no longer R12.1
- net CHG: now also U6.24 (PB3); no longer U6.15 (PB1)
- net DC_OLED: now also U6.14 (PB0); no longer U6.24 (PB3)
- net GND: now also NT3.1
- net GPOUT: now also U6.26 (PB5); no longer U6.18 (PA8)
- net OLED_GPIO_GND: no longer U4.10 (~{WR}), U4.11 (E/~{RD})
- net PGOOD: now also U6.25 (PB4); no longer U6.14 (PB0)
- net XL: now also U6.9 (PA3); no longer U6.7 (PA1)
- net XR: now also U6.6 (PA0); no longer U6.9 (PA3)
- net YD: now also U6.7 (PA1); no longer U6.6 (PA0)
- net ~{CS_ACCEL}: now also U6.10 (PA4); no longer U6.23 (PA15)
- net ~{CS_OLED}: now also U6.18 (PA8); no longer U6.26 (PB5)
- net ~{RES_OLED}: now also U6.15 (PB1); no longer U6.25 (PB4)
- net FT_SCL renamed FT.SCL
- net FT_SDA renamed FT.SDA
- net MCU_RX renamed MCU.RX
- net MCU_TX renamed MCU.TX
- net MISO renamed MCU.MISO
- net MOSI renamed MCU.MOSI
- net SCL renamed MCU.SCL
- net MCU.SCL: now also R12.1; no longer R12.2
- net SCLK renamed MCU.SCLK
- net SDA renamed MCU.SDA
- net SWCLK renamed MCU.SWCLK
- net SWDIO renamed MCU.SWDIO
- new net OLED_GPIO_GND2: NT3.2, U4.10 (~{WR}), U4.11 (E/~{RD})
Other:
- moved on the sheet: C16, C19, C20, R11, R12, R13, R6, R7
